File: Megashield PCB Files/megashield schematic.sch (EAGLE design)
At the start: 1 part

Commit message: adds connectors to schematic file
Parts:
- added J1, J2: RJ11, SparkFun-Connectors:RJ11-6PTH
- added U$1, U$2: 12PIN_TERMINAL_BLOCK, 12pinTerminalBlock:12PIN_TERMINAL_BLOCK
- added U$10, U$11, U$12, U$13, U$9: OSTTC022162_TH, 2pinthruhole:OSTTC022162_TH
- added U$3, U$4, U$5, U$6, U$7, U$8: 4PIN-CONNECTOR4, 4pin connector:4PIN-CONNECTOR4
Changed lines of the file:
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@@
 <layer number="54" name="bGND_GNDA" color="1" fill="9" visible="no" active="no"/>
 <layer number="56" name="wert" color="7" fill="1" visible="no" active="no"/>
+<layer number="57" name="tCAD" color="7" fill="1" visible="no" active="no"/>
+<layer number="59" name="tCarbon" color="7" fill="1" visible="no" active="no"/>
+<layer number="60" name="bCarbon" color="7" fill="1" visible="no" active="no"/>
 <layer number="90" name="Modules" color="5" fill="1" visible="yes" active="yes"/>
 <layer number="91" name="Nets" color="2" fill="1" visible="yes" active="yes"/>
@@
 <layer number="97" name="Info" color="7" fill="1" visible="yes" active="yes"/>
 <layer number="98" name="Guide" color="6" fill="1" visible="yes" active="yes"/>
+<layer number="99" name="SpiceOrder" color="7" fill="1" visible="yes" active="yes"/>
 <layer number="100" name="Muster" color="7" fill="1" visible="no" active="no"/>
 <layer number="101" name="Patch_Top" color="12" fill="4" visible="yes" active="yes"/>
@@
 <layer number="106" name="bPlate" color="7" fill="1" visible="yes" active="yes"/>
 <layer number="107" name="Crop" color="7" fill="1" visible="yes" active="yes"/>
+<layer number="108" name="tplace-old" color="10" fill="1" visible="yes" active="yes"/>
+<layer number="109" name="ref-old" color="11" fill="1" visible="yes" active="yes"/>
+<layer number="110" name="fp0" color="7" fill="1" visible="yes" active="yes"/>
+<layer number="111" name="LPC17xx" color="7" fill="1" visible="yes" active="yes"/>
+<layer number="112" name="tSilk" color="7" fill="1" visible="yes" active="yes"/>
+<layer number="113" name="IDFDebug" color="4" fill="1" visible="yes" active="yes"/>
+<layer number="114" name="Badge_Outline" color="7" fill="1" visible="yes" active="yes"/>
+<layer number="115" name="ReferenceISLANDS" color="7" fill="1" visible="yes" active="yes"/>
 <layer number="116" name="Patch_BOT" color="9" fill="4" visible="yes" active="yes"/>
+<layer number="118" name="Rect_Pads" color="7" fill="1" visible="yes" active="yes"/>
 <layer number="121" name="_tsilk" color="7" fill="1" visible="yes" active="yes"/>
 <layer number="122" name="_bsilk" color="7" fill="1" visible="yes" active="yes"/>
+<layer number="123" name="tTestmark" color="7" fill="1" visible="yes" active="yes"/>
+<layer number="124" name="bTestmark" color="7" fill="1" visible="yes" active="yes"/>
 <layer number="125" name="_tNames" color="7" fill="1" visible="yes" active="yes"/>
+<layer number="126" name="_bNames" color="7" fill="1" visible="yes" active="yes"/>
+<layer number="127" name="_tValues" color="7" fill="1" visible="yes" active="yes"/>
+<layer number="128" name="_bValues" color="7" fill="1" visible="yes" active="yes"/>
+<layer number="129" name="Mask" color="7" fill="1" visible="yes" active="yes"/>
+<layer number="131" name="tAdjust" color="7" fill="1" visible="yes" active="yes"/>
+<layer number="132" name="bAdjust" color="7" fill="1" visible="yes" active="yes"/>
 <layer number="144" name="Drill_legend" color="7" fill="1" visible="yes" active="yes"/>
+<layer number="150" name="Notes" color="7" fill="1" visible="yes" active="yes"/>
 <layer number="151" name="HeatSink" color="7" fill="1" visible="yes" active="yes"/>
+<layer number="152" name="_bDocu" color="7" fill="1" visible="yes" active="yes"/>
+<layer number="153" name="FabDoc1" color="7" fill="1" visible="yes" active="yes"/>
+<layer number="154" name="FabDoc2" color="7" fill="1" visible="yes" active="yes"/>
+<layer number="155" name="FabDoc3" color="7" fill="1" visible="yes" active="yes"/>
+<layer number="199" name="Contour" color="7" fill="1" visible="yes" active="yes"/>
 <layer number="200" name="200bmp" color="1" fill="10" visible="yes" active="yes"/>
 <layer number="201" name="201bmp" color="2" fill="10" visible="yes" active="yes"/>
@@
 <layer number="223" name="223bmp" color="24" fill="1" visible="no" active="no"/>
 <layer number="224" name="224bmp" color="25" fill="1" visible="no" active="no"/>
+<layer number="225" name="225bmp" color="7" fill="1" visible="yes" active="yes"/>
+<layer number="226" name="226bmp" color="7" fill="1" visible="yes" active="yes"/>
+<layer number="227" name="227bmp" color="7" fill="1" visible="yes" active="yes"/>
+<layer number="228" name="228bmp" color="7" fill="1" visible="yes" active="yes"/>
+<layer number="229" name="229bmp" color="7" fill="1" visible="yes" active="yes"/>
+<layer number="230" name="230bmp" color="7" fill="1" visible="yes" active="yes"/>
+<layer number="231" name="231bmp" color="7" fill="1" visible="yes" active="yes"/>
+<layer number="248" name="Housing" color="7" fill="1" visible="yes" active="yes"/>
+<layer number="249" name="Edge" color="7" fill="1" visible="yes" active="yes"/>
 <layer number="250" name="Descript" color="3" fill="1" visible="no" active="no"/>
 <layer number="251" name="SMDround" color="12" fill="11" visible="no" active="no"/>
 <layer number="254" name="cooling" color="7" fill="1" visible="yes" active="yes"/>
+<layer number="255" name="routoute" color="7" fill="1" visible="yes" active="yes"/>
 </layers>
 <schematic xreflabel="%F%N/%S.%C%R" xrefpart="/%S.%C%R">
@@
 <parts>
 <part name="PCB1" library="E14_Arduino_revC" deviceset="ARDUINO_MEGA2560" device=""/>
+<part name="U$1" library="12pinTerminalBlock" deviceset="12PIN_TERMINAL_BLOCK" device=""/>
+<part name="U$2" library="12pinTerminalBlock" deviceset="12PIN_TERMINAL_BLOCK" device=""/>
+<part name="U$3" library="4pin connector" deviceset="4PIN-CONNECTOR" device="4"/>
+<part name="U$4" library="4pin connector" deviceset="4PIN-CONNECTOR" device="4"/>
+<part name="U$5" library="4pin connector" deviceset="4PIN-CONNECTOR" device="4"/>
+<part name="U$6" library="4pin connector" deviceset="4PIN-CONNECTOR" device="4"/>
+<part name="U$7" library="4pin connector" deviceset="4PIN-CONNECTOR" device="4"/>
+<part name="U$8" library="4pin connector" deviceset="4PIN-CONNECTOR" device="4"/>
+<part name="U$9" library="2pinthruhole" deviceset="OSTTC022162_TH" device=""/>
+<part name="U$10" library="2pinthruhole" deviceset="OSTTC022162_TH" device=""/>
+<part name="U$11" library="2pinthruhole" deviceset="OSTTC022162_TH" device=""/>
+<part name="U$12" library="2pinthruhole" deviceset="OSTTC022162_TH" device=""/>
+<part name="U$13" library="2pinthruhole" deviceset="OSTTC022162_TH" device=""/>
+<part name="J1" library="SparkFun-Connectors" deviceset="RJ11-6" device="PTH" value="RJ11"/>
+<part name="J2" library="SparkFun-Connectors" deviceset="RJ11-6" device="PTH" value="RJ11"/>
 </parts>
 <sheets>
@@
 </plain>
 <instances>
-<instance part="PCB1" gate="G$1" x="71.12" y="58.42"/>
+<instance part="PCB1" gate="G$1" x="40.64" y="30.48"/>
+<instance part="U$1" gate="G$1" x="276.86" y="119.38"/>
+<instance part="U$2" gate="G$1" x="215.9" y="119.38"/>
+<instance part="U$3" gate="G$1" x="-147.32" y="114.3"/>
+<instance part="U$4" gate="G$1" x="-66.04" y="114.3"/>
+<instance part="U$5" gate="G$1" x="-147.32" y="81.28"/>
+<instance part="U$6" gate="G$1" x="-66.04" y="81.28"/>
+<instance part="U$7" gate="G$1" x="-147.32" y="48.26"/>
+<instance part="U$8" gate="G$1" x="-66.04" y="48.26"/>
+<instance part="U$9" gate="G$1" x="-187.96" y="-5.08"/>
+<instance part="U$10" gate="G$1" x="-160.02" y="-5.08"/>
+<instance part="U$11" gate="G$1" x="-187.96" y="-27.94"/>
+<instance part="U$12" gate="G$1" x="-160.02" y="-27.94"/>
+<instance part="U$13" gate="G$1" x="-170.18" y="-45.72"/>
+<instance part="J1" gate="G$1" x="185.42" y="-5.08"/>
+<instance part="J2" gate="G$1" x="210.82" y="-5.08"/>
 </instances>
 <busses>
